Commit message: sim0.0.4
urdf 업데이트(그리퍼 추가) 및 mesh 파일 경로 수정

File: irl_dual_arm/urdf/irl_dual_arm.urdf (robot description, URDF)
Before this commit: robot test_robot, 6 links, 5 joints
Links:
- added link gr_rbase, mass 1; collision mesh filename=package://irl_dual_arm/mesh/gripper/r_base.dae scale=1 1 1; visual mesh filename=package://irl_dual_arm/mesh/gripper/r_base.dae scale=1 1 1
- added link r_finger_1_1, mass 1; collision mesh filename=package://irl_dual_arm/mesh/gripper/r_1_1.dae scale=1 1 1; visual mesh filename=package://irl_dual_arm/mesh/gripper/r_1_1.dae scale=1 1 1
- added link r_finger_1_2, mass 1; collision mesh filename=package://irl_dual_arm/mesh/gripper/r_1_2.dae scale=0.001 0.001 0.001; visual mesh filename=package://irl_dual_arm/mesh/gripper/r_1_2.dae scale=0.001 0.001 0.001
- link base: geometry collision mesh filename=package://irl_dual_arm/mesh/arm/base.dae scale=1 1 1; visual mesh filename=package://irl_dual_arm/mesh/arm/base.dae scale=1 1 1
- link link1: geometry collision mesh filename=package://irl_dual_arm/mesh/arm/link1.dae scale=1 1 1; visual mesh filename=package://irl_dual_arm/mesh/arm/link1.dae scale=1 1 1
- link link2: geometry collision mesh filename=package://irl_dual_arm/mesh/arm/link2.dae scale=1 1 1; visual mesh filename=package://irl_dual_arm/mesh/arm/link2.dae scale=1 1 1
- link link3: geometry collision mesh filename=package://irl_dual_arm/mesh/arm/link3.dae scale=1 1 1; visual mesh filename=package://irl_dual_arm/mesh/arm/link3.dae scale=1 1 1
- link link4: geometry collision mesh filename=package://irl_dual_arm/mesh/arm/link4.dae scale=1 1 1; visual mesh filename=package://irl_dual_arm/mesh/arm/link4.dae scale=1 1 1
- link link5: geometry collision mesh filename=package://irl_dual_arm/mesh/arm/link5.dae scale=1 1 1; visual mesh filename=package://irl_dual_arm/mesh/arm/link5.dae scale=1 1 1
Joints:
- added joint joint6: type fixed, parent link5, child gr_rbase, origin xyz=0 0 0.19 rpy=-1.57 -1.57 0
- added joint r_finger1_1: type revolute, parent gr_rbase, child r_finger_1_1, origin xyz=0.0475 -0.002 0.0285 rpy=0 0 0, axis 0 0 1, limit lower=0 upper=0.87 effort=30 velocity=1.571
- added joint r_finger1_2: type revolute, parent r_finger_1_1, child r_finger_1_2, origin xyz=0.05 -0.005 0 rpy=0 0 0, axis 0 0 1, limit lower=0 upper=1.4 effort=30 velocity=1.571, mimic joint=r_finger1_1 multiplier=1.6 offset=0
- joint joint3: origin xyz=0 -0.04 0.03 rpy=1.571 0 0 -> xyz=0 -0.04 0.035 rpy=1.571 0 0
- joint joint4: limit lower=0 upper=1.221 effort=30 velocity=2.093 -> lower=0 upper=1.8 effort=30 velocity=1.571

Commit message: init

File: irl_dual_arm/urdf/irl_dual_arm.urdf (robot description, URDF)
Before this commit: robot test_robot, 6 links, 5 joints
Links:
- added link link6, mass 1; collision box size=0.1 0.1 0.5; visual box size=0.1 0.1 0.5
Joints:
- added joint joint6: type revolute, parent link5, child link6, origin xyz=0 0 0 rpy=0 0 0, axis 0 0 1, limit lower=-1.74 upper=1.74 effort=30 velocity=1.571

Commit message: sim0.1.1
add gripper

File: irl_dual_arm/urdf/irl_dual_arm.urdf (robot description, URDF)
Before this commit: robot IRL_dual_arm, 9 links, 8 joints
Links:
- added link r_finger_2_1, mass 1; collision mesh filename=package://irl_dual_arm/mesh/gripper/r_2_1.dae scale=1 1 1; visual mesh filename=package://irl_dual_arm/mesh/gripper/r_2_1.dae scale=1 1 1
- added link r_finger_2_2, mass 1; collision mesh filename=package://irl_dual_arm/mesh/gripper/r_2_2.dae scale=1 1 1; visual mesh filename=package://irl_dual_arm/mesh/gripper/r_2_2.dae scale=1 1 1
- added link r_finger_3_1, mass 1; collision mesh filename=package://irl_dual_arm/mesh/gripper/r_3_1.dae scale=1 1 1; visual mesh filename=package://irl_dual_arm/mesh/gripper/r_3_1.dae scale=1 1 1
- added link r_finger_3_2, mass 1; collision mesh filename=package://irl_dual_arm/mesh/gripper/r_3_2.dae scale=1 1 1; visual mesh filename=package://irl_dual_arm/mesh/gripper/r_3_2.dae scale=1 1 1
Joints:
- added joint r_finger2_1: type revolute, parent gr_rbase, child r_finger_2_1, origin xyz=0.0475 -0.002 -0.017 rpy=0 0 0, axis 0 0 1, limit lower=0 upper=0.7 effort=30 velocity=1.571
- added joint r_finger2_2: type revolute, parent r_finger_2_1, child r_finger_2_2, origin xyz=0.05 -0.005 0 rpy=0 0 0, axis 0 0 1, limit lower=0 upper=1.4 effort=30 velocity=1.571, mimic joint=r_finger2_1 multiplier=1.6 offset=0
- added joint r_finger3_1: type revolute, parent gr_rbase, child r_finger_3_1, origin xyz=0.0185 0.023 0 rpy=3.14 0 1.57, axis 0 0 1, limit lower=0 upper=0.7 effort=30 velocity=1.571
- added joint r_finger3_2: type revolute, parent r_finger_3_1, child r_finger_3_2, origin xyz=0.05 -0.005 -0.0065 rpy=0 0 0, axis 0 0 1, limit lower=0 upper=1.4 effort=30 velocity=1.571, mimic joint=r_finger3_1 multiplier=1.6 offset=0
- joint r_finger1_1: limit lower=0 upper=0.87 effort=30 velocity=1.571 -> lower=0 upper=0.7 effort=30 velocity=1.571
